File: J-01-Alps.sch (KiCad schematic (older format))
At the start: 17 parts, among them SW1 SW_Push, U1 ATmega32U4-MU, U4 PRTR5V0U2X, Y1 16MHz

Commit message: Cleanup
A few small cleanup updates.
Parts:
- F1: value Polyfuse_Small -> 1A
Changed lines of the file:
@@
 P 1750 3700
 F 0 "F1" V 1545 3700 50  0000 C CNN
-F 1 "Polyfuse_Small" V 1636 3700 50  0000 C CNN
+F 1 "1A" V 1636 3700 50  0000 C CNN
 F 2 "Fuse:Fuse_1206_3216Metric_Pad1.42x1.75mm_HandSolder" H 1800 3500 50  0001 L CNN
 F 3 "~" H 1750 3700 50  0001 C CNN
