File: J-01-Alps.kicad_pcb (KiCad board)
At the start: 2 copper layers, 360.1 x 98.9 mm, 206 parts, among them SW1 SW_Push, U1 ATmega32U4-MU, U4 PRTR5V0U2X, Y1 16MHz

Commit message: Kicad 6 DRC cleanup
Changes to the DRC tool for Kicad 6 required additional cleanup.
Parts:
- F1: value Polyfuse_Small -> 1A
Connections:
- U1 pad 1: Net-(U1-Pad1) -> unconnected-(U1-Pad1)
- U1 pad 12: Net-(U1-Pad12) -> unconnected-(U1-Pad12)
- U1 pad 42: Net-(U1-Pad42) -> unconnected-(U1-Pad42)
Routing:
- net +5V: track 115.7 -> 114.2 mm
- net COL2: track 127.1 -> 125.7 mm
- net XTAL2: track 17.9 -> 17.2 mm

Commit message: Outline adjustment, footprint cleanup
Connections:
- SW-LWIN1 pad 2: Net-(D73-Pad2) -> (no net)
Other:
- outline, holes or cut-outs redrawn

Commit message: PCB dimension verification
Double check of switch positions and edge dimensions.
Parts:
- moved SW-UP1 0.13 mm to (356.4, 137.3)
- moved SW-RIGHT1 0.13 mm to (375.4, 156.4)
- moved SW-DOWN1 0.13 mm to (356.4, 156.4)
- moved SW-LEFT1 0.13 mm to (337.3, 156.4)
Other:
- board size 360.1 x 98.9 mm -> 360 x 98.7 mm

Commit message: Trace cleanup and ISO Enter
Continued trace cleanup for multi-position keys. Added support for three ISO enter orientations - 1.25 vertical and horizontal, and 1.5u vertical.
Parts:
- added SW-ISOEN2: MX_Alps-ISO, Alps_Only:ALPS-1U, F.Cu at (349.2, 104.0)
- added SW-ISOEN3: MX_Alps-ISO, Alps_Only:ALPS-1U, F.Cu at (346.9, 104.0)
- moved D38 4.02 mm to (96.1, 115.9)
- moved D73 2.45 mm to (118.2, 154.0)
- moved D34 1.53 mm to (349.2, 95.3)
- moved C2 1.32 mm to (64.8, 108.5), turned to -90 degrees
- turned SW-3800CAPS1 to 180 degrees
- turned SW-LWIN1 to 180 degrees
Connections:
- SW-LWIN1 pad 2: (no net) -> Net-(D73-Pad2)
Routing:
- net Net-(D38-Pad2): track 8.11 -> 20.5 mm, vias 0 -> 1
- net Net-(D73-Pad2): track 20.0 -> 29.3 mm
- net Net-(D51-Pad2): track 17.0 -> 25.9 mm
- net COL16: track 391.6 -> 385.7 mm
- net COL2: track 125.7 -> 131.3 mm
- net COL15: track 394.7 -> 398.9 mm
- net ROW4: track 430.8 -> 432.8 mm
- net COL12: track 315.8 -> 314.0 mm
- net ROW2: track 391.7 -> 393.4 mm
- net Net-(C2-Pad1): track 3.55 -> 5.15 mm
- net Net-(D78-Pad2): track 17.3 -> 15.7 mm
- net Net-(D34-Pad2): track 5.28 -> 3.76 mm
- net D+: track 97.7 -> 96.3 mm
- net D-: track 99.9 -> 98.5 mm
- net Net-(D55-Pad2): track 17.5 -> 16.2 mm
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
Commit message: Footprint cleanup, add AVR-ISP header footprint
Some cleanup of the bottom row, ISO enter layout, and capslock footprints for more clearance. Addition of the AVR ISP header footprint and mapping to the MCU.
Parts:
- added J1: AVR-ISP-6, Connector_PinHeader_2.54mm:PinHeader_2x03_P2.54mm_Vertical, B.Cu at (67.4, 148.5)
- moved RC3 1.12 mm to (70.5, 135.3), turned to 0 degrees
Connections:
- net Net-(RC3-Pad2) renamed NRST
Routing:
- net ROW1: track 356.4 -> 405.9 mm
- net COL0: track 115.1 -> 156.3 mm
- net ROW2: track 393.4 -> 420.7 mm
- net NRST: track 39.8 -> 59.3 mm
- net +5V: track 114.3 -> 120.2 mm
- net Net-(D74-Pad2): track 19.7 -> 18.6 mm
- net Net-(D16-Pad2): track 17.4 -> 16.5 mm
