File: J-01-Alps.kicad_pcb (KiCad board)
At the start: 2 copper layers, 360 x 98.7 mm, 209 parts, among them J1 AVR-ISP-6, SW1 SW_Push, U1 ATmega32U4-MU, U4 PRTR5V0U2X, Y1 16MHz

Commit message: Silkscreen and edge cut changes, update to .step files
Modified the edge cut profile to be compatible with the upcoming rev2 release of the J-01. Changed silkscreen on front of PCB through-holes to prevent solder from flowing through. Updated Gerbers. Changed 3D models to .step files for export.
Other:
- board size 360 x 98.7 mm -> 360 x 97 mm
